File: Practicas/Practica_1_reguladordevoltaje_tps563200-20200330T234318Z-001/Hardware/_saved_Practica 1 regulador de voltaje tps563200.sch (KiCad schematic (older format))
At the start: 16 parts, among them J1 Screw_Terminal_01x02, J2 Screw_Terminal_01x02, U1 TPS563200

Commit message: P1 Version 2.0: se realizo el ruteado con el uso de los planos, escribir texto e insertar logos o simbologia en forma de huellas
Parts:
- gave numbers to parts that had none: 4
Changed lines of the file:
@@
 	7150 2850 7225 2850
 $Comp
-L Mechanical:MountingHole_Pad MH?
+L Mechanical:MountingHole_Pad MH1
 U 1 1 5E8B70B5
 P 4050 3975
-F 0 "MH?" H 4150 3980 50  0000 L CNN
+F 0 "MH1" H 4150 3980 50  0000 L CNN
 F 1 "MountingHole_Pad" H 4150 3935 50  0001 L CNN
 F 2 "MountingHole:MountingHole_3.2mm_M3_DIN965_Pad" H 4050 3975 50  0001 C CNN
@@
 $EndComp
 $Comp
-L power:GND #PWR?
+L power:GND #PWR0115
 U 1 1 5E8B7169
 P 4050 4125
-F 0 "#PWR?" H 4050 3875 50  0001 C CNN
+F 0 "#PWR0115" H 4050 3875 50  0001 C CNN
 F 1 "GND" H 4055 3952 50  0001 C CNN
 F 2 "" H 4050 4125 50  0001 C CNN
@@
 	4050 4075 4050 4125
 $Comp
-L Mechanical:MountingHole_Pad MH?
+L Mechanical:MountingHole_Pad MH2
 U 1 1 5E8BB459
 P 4400 3975
-F 0 "MH?" H 4500 3980 50  0000 L CNN
+F 0 "MH2" H 4500 3980 50  0000 L CNN
 F 1 "MountingHole_Pad" H 4500 3935 50  0001 L CNN
 F 2 "MountingHole:MountingHole_3.2mm_M3_DIN965_Pad" H 4400 3975 50  0001 C CNN
@@
 $EndComp
 $Comp
-L power:GND #PWR?
+L power:GND #PWR0116
 U 1 1 5E8BB460
 P 4400 4125
-F 0 "#PWR?" H 4400 3875 50  0001 C CNN
+F 0 "#PWR0116" H 4400 3875 50  0001 C CNN
 F 1 "GND" H 4405 3952 50  0001 C CNN
 F 2 "" H 4400 4125 50  0001 C CNN
@@
 	4400 4075 4400 4125
 $Comp
-L Mechanical:MountingHole_Pad MH?
+L Mechanical:MountingHole_Pad MH3
 U 1 1 5E8BBB76
 P 4750 3975
-F 0 "MH?" H 4850 3980 50  0000 L CNN
+F 0 "MH3" H 4850 3980 50  0000 L CNN
 F 1 "MountingHole_Pad" H 4850 3935 50  0001 L CNN
 F 2 "MountingHole:MountingHole_3.2mm_M3_DIN965_Pad" H 4750 3975 50  0001 C CNN
@@
 $EndComp
 $Comp
-L power:GND #PWR?
+L power:GND #PWR0117
 U 1 1 5E8BBB7D
 P 4750 4125
-F 0 "#PWR?" H 4750 3875 50  0001 C CNN
+F 0 "#PWR0117" H 4750 3875 50  0001 C CNN
 F 1 "GND" H 4755 3952 50  0001 C CNN
 F 2 "" H 4750 4125 50  0001 C CNN
@@
 	4750 4075 4750 4125
 $Comp
-L Mechanical:MountingHole_Pad MH?
+L Mechanical:MountingHole_Pad MH4
 U 1 1 5E8BC307
 P 5075 3975
-F 0 "MH?" H 5175 3980 50  0000 L CNN
+F 0 "MH4" H 5175 3980 50  0000 L CNN
 F 1 "MountingHole_Pad" H 5175 3935 50  0001 L CNN
 F 2 "MountingHole:MountingHole_3.2mm_M3_DIN965_Pad" H 5075 3975 50  0001 C CNN
@@
 $EndComp
 $Comp
-L power:GND #PWR?
+L power:GND #PWR0118
 U 1 1 5E8BC30E
 P 5075 4125
-F 0 "#PWR?" H 5075 3875 50  0001 C CNN
+F 0 "#PWR0118" H 5075 3875 50  0001 C CNN
 F 1 "GND" H 5080 3952 50  0001 C CNN
 F 2 "" H 5075 4125 50  0001 C CNN
